Commit message: added readme, other tweaks

File: navviswimu.urdf (robot description, URDF)
Before this commit: robot Navvis, 10 links, 9 joints
Links:
- added link base_link
- added link imu; collision sphere radius=0.1; visual sphere radius=0.1
Joints:
- added joint base_imu_joint: type fixed, parent base_link, child imu, origin xyz=0.0 0.0 0.0 rpy=3.1405788 0.0034281 3.1382064
- added joint base_link_base_joint: type fixed, parent base_link, child base, origin xyz=0.07 0 1.792 rpy=0.0 3.14159265359 0.0
